File: XilinxXC95xxxDevBoard.kicad_pcb (KiCad board)
At the start: 4 copper layers, 100 x 100 mm, 55 parts, among them J1 USB_B_Micro, J10 Conn_02x13_Odd_Even, J11 U3Bank1, J12 U3Bank2, J13 U3Bank3, J14 U3Bank4, J2 Conn_02x06_Odd_Even, J3 JTAG, J4 Conn_02x06_Odd_Even, J5 Conn_02x06_Odd_Even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

Commit message: refine labelling
Parts:
- added C15: 10uF, Capacitor_SMD:C_0603_1608Metric, F.Cu at (35.5, 90.1)
- added QR*****: ProjectLink, Library:ProjectLink, F.Cu at (53.6, 45.6)
- added QR*****: https://github.com/jimbro1000/XilinxXC95xxxDevBoard, Library:ProjectLink, B.Cu at (80.0, 94.3)
- C7, C8: footprint Capacitor_THT:C_Disc_D3.0mm_W1.6mm_P2.50mm -> Capacitor_SMD:C_0603_1608Metric
- SW1: value SW_SPST -> OS102011MA1QN1; footprint Library:SWITCH_03211B -> Library:OS102011MA1QN1_CNK
- moved C7 37.9 mm to (57.3, 97.9), turned to 0 degrees
- moved C8 16.4 mm to (41.0, 83.8), turned to 90 degrees
- moved SW1 11.4 mm to (117.8, 106.5), turned to 90 degrees
- moved J4 1.12 mm to (114.7, 81.1)
- moved C5 1.12 mm to (114.6, 65.3)
- moved J5 0.54 mm to (87.8, 68.5)
- moved C3 0.54 mm to (87.8, 84.2)
Routing:
- net +5V: track 63.0 -> 74.8 mm
- net Net-(J1-VBUS): track 7.42 -> 15.7 mm
- net /U2VCC: track 14.2 -> 19.3 mm
- net GND: track 12.2 -> 15.1 mm, vias 18 -> 26
- net /U1MB16: track 7.55 -> 8.67 mm
- net /U1M17: track 7.93 -> 9.06 mm
- net /U1MB14: track 7.21 -> 8.34 mm
- net /U1MB12: track 7.83 -> 8.95 mm
- net /U1MB13: track 4.34 -> 5.47 mm
- net /U1MB17: track 4.77 -> 5.89 mm
- net /U1MB15: track 4.38 -> 5.50 mm
- net /U1VIO: track 49.6 -> 50.2 mm
- net /U1M1: track 8.38 -> 8.92 mm
- net /U1MB1: track 5.51 -> 6.05 mm
- net /U1M2: track 5.12 -> 5.66 mm
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Other:
- board text added: "A1 B1"
- board text added: "A10 A11"
- board text added: "A12 A13"
- board text added: "A14 A15"
- board text added: "A16 NC"
- board text added: "A4 A2"
- board text added: "A6 CL3"
- board text added: "A9 A8"
- board text added: "B10 B11"
- board text added: "B13 B14"
- board text added: "B15 B16"
- board text added: "B17 A17"
- board text added: "B2 B4"
- board text added: "B8 B9"
- board text added: "CK1 P20"
- board text added: "CK3 P28"
- board text added: "CL1 CL2"
- board text added: "GND Vcc"
- board text added: "GND Vio"
- board text added: "GSR B7"
- board text added: "NC B12"
- board text added: "NC NC"
- board text added: "NC P25"
- board text added: "P11 P10"
- board text added: "P13 P12"
- board text added: "P15 P14"
- board text added: "P17 P16"
- board text added: "P19 P18"
- board text added: "P24 CK2"
- board text added: "P29 P30"
- board text added: "P32 P33"
- board text added: "P34 P35"
- board text added: "P36 P37"
- board text added: "P39 P40"
- board text added: "P41 P42"
- board text added: "P43 P46"
- board text added: "P49 P50"
- board text added: "P52 P53"
- board text added: "P54 P55"
- board text added: "P56 P58"
- board text added: "P59 P60"
- board text added: "P61 P63"
- board text added: "P64 P65"
- board text added: "P66 P67"
- board text added: "P68 P70"
- board text added: "P7 P6"
- board text added: "P71 P72"
- board text added: "P73 P74"
- board text added: "P76 P77"
- board text added: "P78 P79"
- board text added: "P80 P81"
- board text added: "P82 P85"
- board text added: "P86 P87"
- board text added: "P89 P90"
- board text added: "P9 P8"
- board text added: "P91 P92"
- board text added: "P93 P94"
- board text added: "P95 P96"
- board text added: "P97 GSR"
- board text added: "TS1 TS2"
- board text added: "TS2 TS1"
- board text added: "TS4 TS3"
- board text added: "Vcc GND"
