File: XilinxXC95xxxDevBoard.kicad_sch (KiCad schematic)
At the start: 55 parts, among them J1 USB_B_Micro, J10 Conn_02x13_Odd_Even, J11 U3Bank1, J12 U3Bank2, J13 U3Bank3, J14 U3Bank4, J2 Conn_02x06_Odd_Even, J3 JTAG, J4 Conn_02x06_Odd_Even, J5 Conn_02x06_Odd_Even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

Commit message: refine labelling
Parts:
- removed SW1: SW_SPST, Library:SWITCH_03211B, symbol Switch:SW_SPST
- added C15: 10uF, Capacitor_SMD:C_0603_1608Metric, symbol Device:C_Small
- added SW1: OS102011MA1QN1, Library:OS102011MA1QN1_CNK, symbol Library:OS102011MA1QN1
- C1, C2: LCSC (none) -> C13585
- C11, C12, C13, C14: LCSC (none) -> C19702
- C7, C8: footprint Capacitor_THT:C_Disc_D3.0mm_W1.6mm_P2.50mm -> Capacitor_SMD:C_0603_1608Metric; LCSC (none) -> C19702
- D1, D2, D3, D4, D5: LCSC (none) -> C2297
- H1, H2, H3, H4, J10, J11, J12, J13, J14, J2, J3, J4, J5, J6, J7, J8, J9, JP4, JP5, JP6: now not fitted
- J1: LCSC (none) -> C2894326
- JP1, JP2, JP3: now not fitted; now in the parts list
- P1: now not fitted; now left out of the parts list
- R1, R2, R3, R4, R5: LCSC (none) -> C23138
- U3: LCSC (none) -> C500874
- U4: LCSC (none) -> C7432020
Connections:
- net +5V: now also SW1.3
- net GND: now also C15.2
- net U2VCC: now also C15.1
- net at J1.1 (VBUS): now also SW1.1
- no-connect marks 34 -> 35
Other:
- moved on the sheet: C1, C2, D1, D2, J1, L1, R1, R2, U4
